File: circuits/video_output_stage/video_output_stage.sch (KiCad schematic (older format))
At the start: 20 parts

Commit message: generated netlist; have actual transistor
Parts:
- added Q1: C5468, symbol Q_NPN_CBE
- TR6: renamed from TR06; value INDUCTOR -> 20uH
- gave numbers to parts that had none: 2
Connections:
- net T_1: no longer names the net of R69.1, R70.1, R72.1
- net T_1: now also Q1.1 (C)
- net T_2: no longer names the net of TR6.1
- net T_2: now also Q1.2 (B)
- net T_3: no longer names the net of R26.2, R27.2, R28.1, R29.2, R71.2
- net T_3: now also Q1.3 (E)
Changed lines of the file:
@@
 LIBS:contrib
 LIBS:valves
+LIBS:video_output_stage-cache
 EELAYER 25 0
 EELAYER END
@@
 VIDEO_OUT
 $Comp
-L CONN_01X07 P?
+L CONN_01X07 P1
 U 1 1 58E7F12A
 P 1700 3800
-F 0 "P?" H 1700 4200 50  0000 C CNN
+F 0 "P1" H 1700 4200 50  0000 C CNN
 F 1 "CONN_01X07" V 1800 3800 50  0000 C CNN
 F 2 "" H 1700 3800 50  0000 C CNN
@@
 $EndComp
 $Comp
-L GND #PWR?
+L GND #PWR2
 U 1 1 58E7F295
 P 2350 3800
-F 0 "#PWR?" H 2350 3550 50  0001 C CNN
+F 0 "#PWR2" H 2350 3550 50  0001 C CNN
 F 1 "GND" H 2350 3650 50  0000 C CNN
 F 2 "" H 2350 3800 50  0000 C CNN
@@
 	1    0    0    -1
 $EndComp
-Text GLabel 3000 2250 1    60   Input ~ 0
-T_1
-Text GLabel 3200 2250 1    60   Input ~ 0
-T_2
-Text GLabel 3400 2250 1    60   Input ~ 0
-T_3
 $Comp
 L C C18
@@
 $EndComp
 $Comp
-L GND #PWR?
+L GND #PWR1
 U 1 1 58E7F98A
 P 2000 4650
-F 0 "#PWR?" H 2000 4400 50  0001 C CNN
+F 0 "#PWR1" H 2000 4400 50  0001 C CNN
 F 1 "GND" H 2000 4500 50  0000 C CNN
 F 2 "" H 2000 4650 50  0000 C CNN
@@
 $EndComp
 $Comp
-L GND #PWR?
+L GND #PWR3
 U 1 1 58E7FC8D
 P 2350 4650
-F 0 "#PWR?" H 2350 4400 50  0001 C CNN
+F 0 "#PWR3" H 2350 4400 50  0001 C CNN
 F 1 "GND" H 2350 4500 50  0000 C CNN
 F 2 "" H 2350 4650 50  0000 C CNN
@@
 $EndComp
 $Comp
-L 74HC04 U?
+L 74HC04 M3
 U 3 1 58E80266
 P 4350 4000
-F 0 "U?" H 4500 4100 50  0000 C CNN
+F 0 "M3" H 4500 4100 50  0000 C CNN
 F 1 "74HC04" H 4550 3900 50  0000 C CNN
 F 2 "" H 4350 4000 50  0000 C CNN
@@
 $EndComp
 $Comp
-L 74HC04 U?
+L 74HC04 M3
 U 4 1 58E806AD
 P 4350 3650
-F 0 "U?" H 4500 3750 50  0000 C CNN
+F 0 "M3" H 4500 3750 50  0000 C CNN
 F 1 "74HC04" H 4550 3550 50  0000 C CNN
 F 2 "" H 4350 3650 50  0000 C CNN
@@
 $EndComp
 $Comp
-L 74HC04 U?
+L 74HC04 M3
 U 5 1 58E8079D
 P 4350 3300
-F 0 "U?" H 4500 3400 50  0000 C CNN
+F 0 "M3" H 4500 3400 50  0000 C CNN
 F 1 "74HC04" H 4550 3200 50  0000 C CNN
 F 2 "" H 4350 3300 50  0000 C CNN
@@
 $EndComp
 $Comp
-L 74HC04 U?
+L 74HC04 M3
 U 6 1 58E80834
 P 4350 2950
-F 0 "U?" H 4500 3050 50  0000 C CNN
+F 0 "M3" H 4500 3050 50  0000 C CNN
 F 1 "74HC04" H 4550 2850 50  0000 C CNN
 F 2 "" H 4350 2950 50  0000 C CNN
@@
 	1900 2500 2100 2500
 Wire Wire Line
-	2400 2500 3000 2500
-Wire Wire Line
-	3000 2500 3000 2250
+	3000 2500 2400 2500
+Wire Wire Line
+	3000 2150 3000 2500
 Wire Wire Line
 	2600 2600 2600 2500
@@
 Connection ~ 3200 3300
 Wire Wire Line
-	3400 2250 3400 2750
+	3400 2150 3400 2750
 Wire Wire Line
 	3400 2750 3200 2750
@@
 Connection ~ 6050 2950
 $Comp
-L INDUCTOR TR06
+L INDUCTOR TR6
 U 1 1 58E81614
 P 3900 2450
-F 0 "TR06" V 3850 2450 50  0000 C CNN
-F 1 "INDUCTOR" V 4000 2450 50  0000 C CNN
+F 0 "TR6" V 3850 2450 50  0000 C CNN
+F 1 "20uH" V 4000 2450 50  0000 C CNN
 F 2 "" H 3900 2450 50  0000 C CNN
 F 3 "" H 3900 2450 50  0000 C CNN
@@
 $EndComp
 $Comp
-L +5V #PWR?
+L +5V #PWR4
 U 1 1 58E81681
 P 4400 2450
-F 0 "#PWR?" H 4400 2300 50  0001 C CNN
+F 0 "#PWR4" H 4400 2300 50  0001 C CNN
 F 1 "+5V" H 4400 2590 50  0000 C CNN
 F 2 "" H 4400 2450 50  0000 C CNN
@@
 	4200 2450 4400 2450
 Wire Wire Line
-	3600 2450 3200 2450
-Wire Wire Line
-	3200 2450 3200 2250
+	3200 2450 3600 2450
+$Comp
+L Q_NPN_CBE Q1
+U 1 1 58EB8E62
+P 3200 2250
+F 0 "Q1" H 3500 2300 50  0000 R CNN
+F 1 "C5468" H 3800 2200 50  0000 R CNN
+F 2 "" H 3400 2350 50  0000 C CNN
+F 3 "" H 3200 2250 50  0000 C CNN
+	1    3200 2250
+	0    -1   -1   0
+$EndComp
 $EndSCHEMATC

Commit message: fixing 7805 symbol initial PCB layout quickly giving up on kicad
Parts:
- added P2: CONN_01X05, Pin_Headers:Pin_Header_Straight_1x05, symbol CONN_01X05
- added P3: BNC, Connect:PINHEAD1-2, symbol BNC
- added U1: 7805, TO_SOT_Packages_THT:TO-220_Neutral123_Vertical_LargePads, symbol 7805
- C18, C53: footprint (none) -> Capacitors_ThroughHole:C_Disc_D6_P5
- D7, D8, D9: footprint (none) -> Diodes_ThroughHole:Diode_DO-35_SOD27_Horizontal_RM10
- M3: footprint (none) -> Housings_DIP:DIP-14_W7.62mm_LongPads
- P1: footprint (none) -> Connectors_Phoenix:PhoenixContact_MSTBVA-G_07x5.00mm_Vertical
- Q1: footprint (none) -> TO_SOT_Packages_THT:TO-92_Inline_Wide
- R26, R27, R28, R29, R67, R69, R70, R71, R72: footprint (none) -> Resistors_ThroughHole:Resistor_Horizontal_RM15mm
- TR6: footprint (none) -> Choke_Axial_ThroughHole:Choke_Horizontal_RM20mm
Connections:
- net VCC is gone; now on net +5V: M3.14 (VCC), M3.14 (VCC), M3.14 (VCC), M3.14 (VCC)
- net +5V: now also P2.4 (P4), U1.3 (VO)
- net CH_BLUE: now also P2.1 (P1)
- net CH_GREEN: now also P2.2 (P2)
- net CH_RED: now also P2.3 (P3)
- net GND: now also P2.5 (P5), P3.2 (Ext), U1.2 (GND)
- net VIDEO_OUT: now also P3.1 (In)
- net VIN: now reaches P1.6 (P6)
- net VIN: now also U1.1 (VI)

Commit message: circuit's pretty much done; now for a new board
Parts:
- added C?: 100nF, Capacitors_ThroughHole:C_Disc_D6_P5, symbol C
- added C?: 10nF, Capacitors_ThroughHole:C_Disc_D6_P5, symbol C
- added D? (x3): 1N4148, Diodes_ThroughHole:Diode_DO-35_SOD27_Horizontal_RM10, symbol D
- added M? (x4): 74HC04, Housings_DIP:DIP-14_W7.62mm_LongPads, symbol 74HC04
- added P?: CONN_01X07, Connectors_Phoenix:PhoenixContact_MSTBVA-G_07x5.00mm_Vertical, symbol CONN_01X07
- added P?: CONN_01X05, Pin_Headers:Pin_Header_Straight_1x05, symbol CONN_01X05
- added P?: BNC, Connect:PINHEAD1-2, symbol BNC
- added Q?: C5468, TO_SOT_Packages_THT:TO-92_Inline_Wide, symbol Q_NPN_CBE
- added R?: 100, Resistors_ThroughHole:Resistor_Horizontal_RM15mm, symbol R
- added R? (x2): 2.4K, Resistors_ThroughHole:Resistor_Horizontal_RM15mm, symbol R
- added R?: 1.2K, Resistors_ThroughHole:Resistor_Horizontal_RM15mm, symbol R
- added R?: 1.8K, Resistors_ThroughHole:Resistor_Horizontal_RM15mm, symbol R
- added R?: 460, Resistors_ThroughHole:Resistor_Horizontal_RM15mm, symbol R
- added R?: 1K, Resistors_ThroughHole:Resistor_Horizontal_RM15mm, symbol R
- added R?: 620, Resistors_ThroughHole:Resistor_Horizontal_RM15mm, symbol R
- added R?: 670, Resistors_ThroughHole:Resistor_Horizontal_RM15mm, symbol R
- added TR?: 20uH, Choke_Axial_ThroughHole:Choke_Horizontal_RM20mm, symbol INDUCTOR
- added U?: 7805, TO_SOT_Packages_THT:TO-220_Neutral123_Vertical_LargePads, symbol 7805
Connections:
- net +5V: now also M?.14 (VCC), M?.14 (VCC), M?.14 (VCC), M?.14 (VCC), P?.4 (P4), TR?.2, U?.3 (VO)
- net CH_BLUE: now also D?.2 (A), M?.1, P?.1 (P1)
- net CH_GREEN: now also D?.2 (A), M?.1, P?.2 (P2)
- net CH_RED: now also D?.2 (A), M?.1, P?.3 (P3)
- net GND: now also C?.1, C?.2, M?.7 (GND), M?.7 (GND), M?.7 (GND), M?.7 (GND), P?.2 (Ext), P?.4 (P4), P?.5 (P5), U?.2 (GND)
- net VIDEO_OUT: now also P?.1 (In), R?.2
- net VIN: now also P?.6 (P6), U?.1 (VI)
- net at C18.2, P1.1 (P1), R69.2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: now also C?.2, P?.1 (P1), R?.2, R?.2
- net at C53.1, P1.2 (P2), R71.1: now also C?.1, P?.2 (P2), R?.1
- net at P1.3 (P3): now also P?.3 (P3)
- net at P1.5 (P5): now also P?.5 (P5)
- net at P1.7 (P7): now also P?.7 (P7)
- net at Q1.1 (C), R69.1, R70.1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: now also Q?.1 (C), R?.1, R?.1, R?.1
- net at Q1.3 (E), R26.2, R27.2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: now also Q?.3 (E), R?.1, R?.2, R?.2, R?.2, R?.2
- net at M3.12, R27.1: now also M?.2, R?.1
- net at M3.10, R28.2: now also M?.2, R?.2
- net at M3.8, R29.1: now also M?.2, R?.1
- net at M3.6, R26.1: now also M?.2, R?.1
- net at M3.5, R67.2: now also M?.1, R?.2
- net at D7.1 (K), D8.1 (K), D9.1 (K)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: now also D?.1 (K), D?.1 (K), D?.1 (K), R?.1
- net at Q1.2 (B), TR6.1: now also Q?.2 (B), TR?.1
